Commit message: Add placeholders for the front & rear face sensor mounts

File: clearpath_platform_description/urdf/a300/attachments/observer_backpack.urdf.xacro (robot description, xacro)
@@ -51,4 +51,16 @@
       <origin xyz="0 0 0.4" rpy="0 0 0" />
     </joint>
+    <link name="${name}_front_face_mount" />
+    <joint name="${name}_front_face_link" type="fixed">
+      <parent link="${name}_center_mount" />
+      <child link="${name}_front_face_mount" />
+      <origin xyz="0.33 0 -0.08" rpy="0 0 0" />
+    </joint>
+    <link name="${name}_rear_face_mount" />
+    <joint name="${name}_rear_face_link" type="fixed">
+      <parent link="${name}_center_mount" />
+      <child link="${name}_rear_face_mount" />
+      <origin xyz="-0.33 0 -0.08" rpy="0 0 3.1459" />
+    </joint>
   </xacro:macro>
 </robot>
