Commit message: Add sensor mount points from Rhys

File: clearpath_platform_description/urdf/a300/attachments/observer_arch.urdf.xacro (robot description, xacro)
@@ -27,17 +27,36 @@
     <!--
         Sensor mounting points
-        TODO: get these measurements from Rhys
     -->
     <link name="${name}_left_antenna_mount" />
-    <joint name="${name}_left_antenna_joint" type="fixed">
+    <joint name="${name}_left_antenna_mount_joint" type="fixed">
       <parent link="${name}_link" />
       <child link="${name}_left_antenna_mount" />
-      <origin xyz="0 0.26 0.45" rpy="0 0 0" />
+      <origin xyz="0 0.260 0.44536" rpy="0 0 0" />
     </joint>
     <link name="${name}_right_antenna_mount" />
-    <joint name="${name}_right_antenna_joint" type="fixed">
+    <joint name="${name}_right_antenna_mount_joint" type="fixed">
       <parent link="${name}_link" />
       <child link="${name}_right_antenna_mount" />
-      <origin xyz="0 -0.26 0.45" rpy="0 0 0" />
+      <origin xyz="0 -0.260 0.44536" rpy="0 0 0" />
+    </joint>
+    <link name="${name}_lidar_mount" />
+    <joint name="${name}_lidar_mount_joint" type="fixed">
+      <parent link="${name}_link" />
+      <child link="${name}_lidar_mount" />
+      <origin xyz="0.130 0 0.30256" rpy="3.14159 0 0" />
+    </joint>
+    <!-- front-facing camera suspended under sensor arch -->
+    <link name="${name}_front_camera_mount" />
+    <joint name="${name}_front_camera_mount_joint" type="fixed">
+      <parent link="${name}_link" />
+      <child link="${name}_front_camera_mount" />
+      <origin xyz="0.055 0 0.40896" rpy="3.14159 0 0" />
+    </joint>
+    <!-- rear-facing camera suspended under sensor arch -->
+    <link name="${name}_front_camera_mount" />
+    <joint name="${name}_front_camera_mount_joint" type="fixed">
+      <parent link="${name}_link" />
+      <child link="${name}_front_camera_mount" />
+      <origin xyz="-0.071992 0 0.4036838" rpy="0 -0.6021385919380436 3.14159" />
     </joint>
   </xacro:macro>

File: clearpath_platform_description/urdf/a300/attachments/observer_backpack.urdf.xacro (robot description, xacro)
@@ -45,21 +45,31 @@
         Mount points for sensors, other accessories
     -->
+    <!-- center of the adjustable track on top -->
     <link name="${name}_center_mount" />
     <joint name="${name}_center_joint" type="fixed">
       <parent link="${name}_enclosure_link" />
       <child link="${name}_center_mount" />
-      <origin xyz="0 0 0.4" rpy="0 0 0" />
+      <origin xyz="0 0 0.4074593" rpy="0 0 0" />
     </joint>
-    <link name="${name}_front_face_mount" />
-    <joint name="${name}_front_face_link" type="fixed">
-      <parent link="${name}_center_mount" />
-      <child link="${name}_front_face_mount" />
-      <origin xyz="0.33 0 -0.08" rpy="0 0 0" />
+    <!-- standard rear-mounted antennas -->
+    <link name="${name}_antenna_mount" />
+    <joint name="${name}_antenna_mount_link" type="fixed">
+      <parent link="${name}_enclosure_link" />
+      <child link="${name}_antenna_mount" />
+      <origin xyz="-0.4028 0 0.4074593" rpy="0 0 0" />
     </joint>
-    <link name="${name}_rear_face_mount" />
-    <joint name="${name}_rear_face_link" type="fixed">
-      <parent link="${name}_center_mount" />
-      <child link="${name}_rear_face_mount" />
-      <origin xyz="-0.33 0 -0.08" rpy="0 0 3.1459" />
+    <!-- rear-mounted fixposition -->
+    <link name="${name}_ins_mount" />
+    <joint name="${name}_ins_mouint_link" type="fixed">
+      <parent link="${name}_enclosure_link" />
+      <child link="${name}_ins_mount" />
+      <origin xyz="-0.4 0.0 0.3192593" rpy="3.14159 0 0" />
+    </joint>
+    <!-- front-mounted robin -->
+    <link name="${name}_front_lidar_mount" />
+    <joint name="${name}_front_lidar_mount_link" type="fixed">
+      <parent link="${name}_enclosure_link" />
+      <child link="${name}_front_lidar_mount" />
+      <origin xyz="0.40 0 0.2708593" rpy="0 0 0" />
     </joint>
   </xacro:macro>

Commit message: Fix the angle of the rear camera mount, rear INS. Remove duplicate link name

File: clearpath_platform_description/urdf/a300/attachments/observer_arch.urdf.xacro (robot description, xacro)
@@ -54,9 +54,9 @@
     </joint>
     <!-- rear-facing camera suspended under sensor arch -->
-    <link name="${name}_front_camera_mount" />
-    <joint name="${name}_front_camera_mount_joint" type="fixed">
+    <link name="${name}_rear_camera_mount" />
+    <joint name="${name}_rear_camera_mount_joint" type="fixed">
       <parent link="${name}_link" />
-      <child link="${name}_front_camera_mount" />
-      <origin xyz="-0.071992 0 0.4036838" rpy="0 -0.6021385919380436 3.14159" />
+      <child link="${name}_rear_camera_mount" />
+      <origin xyz="-0.071992 0 0.4036838" rpy="0 0.6021385919380436 3.14159" />
     </joint>
   </xacro:macro>

File: clearpath_platform_description/urdf/a300/attachments/observer_backpack.urdf.xacro (robot description, xacro)
@@ -64,5 +64,5 @@
       <parent link="${name}_enclosure_link" />
       <child link="${name}_ins_mount" />
-      <origin xyz="-0.4 0.0 0.3192593" rpy="3.14159 0 0" />
+      <origin xyz="-0.4 0.0 0.3192593" rpy="3.14159 0 3.14159" />
     </joint>
     <!-- front-mounted robin -->

Commit message: Add spotlight attachment with light plugin for simulation

File: clearpath_platform_description/urdf/a300/attachments/observer_arch.urdf.xacro (robot description, xacro)
@@ -51,5 +51,5 @@
       <parent link="${name}_link" />
       <child link="${name}_front_camera_mount" />
-      <origin xyz="0.055 0 0.40896" rpy="3.14159 0 0" />
+      <origin xyz="0.0775 0 0.40896" rpy="0 0 0" />
     </joint>
     <!-- rear-facing camera suspended under sensor arch -->
@@ -58,5 +58,30 @@
       <parent link="${name}_link" />
       <child link="${name}_rear_camera_mount" />
-      <origin xyz="-0.071992 0 0.4036838" rpy="0 0.6021385919380436 3.14159" />
+      <origin xyz="-0.09053483924399536 0 0.39093965966919125" rpy="0 0.6021385919380436 3.14159" />
+    </joint>
+    <!-- corner mounts for lights, etc... -->
+    <link name="${name}_front_left_corner_mount" />
+    <joint name="${name}_front_left_corner_mount_joint" type="fixed">
+      <parent link="${name}_link" />
+      <child link="${name}_front_left_corner_mount" />
+      <origin xyz="0.07 0.310 0.44536" rpy="0 0 0" />
+    </joint>
+    <link name="${name}_front_right_corner_mount" />
+    <joint name="${name}_front_right_corner_mount_joint" type="fixed">
+      <parent link="${name}_link" />
+      <child link="${name}_front_right_corner_mount" />
+      <origin xyz="0.07 -0.310 0.44536" rpy="0 0 0" />
+    </joint>
+    <link name="${name}_rear_left_corner_mount" />
+    <joint name="${name}_rear_left_corner_mount_joint" type="fixed">
+      <parent link="${name}_link" />
+      <child link="${name}_rear_left_corner_mount" />
+      <origin xyz="-0.07 0.310 0.44536" rpy="0 0 3.14159" />
+    </joint>
+    <link name="${name}_rear_right_corner_mount" />
+    <joint name="${name}_rear_right_corner_mount_joint" type="fixed">
+      <parent link="${name}_link" />
+      <child link="${name}_rear_right_corner_mount" />
+      <origin xyz="-0.07 -0.310 0.44536" rpy="0 0 3.14159" />
     </joint>
   </xacro:macro>
