Commit message: Add the ability to specify the OS-1 cap type & omit the base plate

File: clearpath_sensors_description/urdf/ouster_os1.urdf.xacro (robot description, xacro)
@@ -19,4 +19,5 @@
     parent_link
     cap:=halo
+    base:=base
     *origin
     samples_h:=1024 min_ang_h:=${-pi} max_ang_h:=${pi}
@@ -28,7 +29,14 @@
     <xacro:property name="lidar_height" value="0.05835"/>
     <xacro:property name="lidar_diameter" value="0.087"/>
-    <xacro:property name="base_mass" value="0."/>
-    <xacro:property name="base_height" value="0.0225"/>
-    <xacro:property name="base_length" value="0.110"/>
+    <xacro:if value="${base == 'base'}">
+      <xacro:property name="base_mass" value="0."/>
+      <xacro:property name="base_height" value="0.0225"/>
+      <xacro:property name="base_length" value="0.110"/>
+    </xacro:if>
+    <xacro:unless value="${base == 'base'}">
+      <xacro:property name="base_mass" value="0."/>
+      <xacro:property name="base_height" value="0."/>
+      <xacro:property name="base_length" value="0."/>
+    </xacro:unless>
     <xacro:property name="fins_mass" value="0.079"/>
     <xacro:property name="fins_height" value="0.022"/>
@@ -38,31 +46,36 @@
     <xacro:property name="halo_diameter" value="0.08679"/>
     <!-- Base Link -->
-    <link name="${name}_base_link">
-      <inertial>
-        <mass value="${base_mass}"/>
-        <origin xyz="0 0 ${base_height/2}"/>
-        <xacro:ouster_box_inertia
-          mass="${base_mass}"
-          x="${base_length}"
-          y="${base_length}"
-          z="${base_height}"
-        />
-      </inertial>
-      <visual>
-        <material name="ouster_grey">
-          <color rgba="0.8 0.8 0.8 1.0"/>
-        </material>
-        <origin xyz="0 0 ${base_height}"/>
-        <geometry>
-          <mesh filename="package://clearpath_sensors_description/meshes/ouster/os1_base.dae"/>
-        </geometry>
-      </visual>
-      <collision>
-        <origin xyz="0 0 ${base_height/2}"/>
-        <geometry>
-          <box size="${base_length} ${base_length} ${base_height}"/>
-        </geometry>
-      </collision>
+    <xacro:if value="${base == 'base'}">
+      <link name="${name}_base_link">
+        <inertial>
+          <mass value="${base_mass}"/>
+          <origin xyz="0 0 ${base_height/2}"/>
+          <xacro:ouster_box_inertia
+            mass="${base_mass}"
+            x="${base_length}"
+            y="${base_length}"
+            z="${base_height}"
+          />
+        </inertial>
+        <visual>
+          <material name="ouster_grey">
+            <color rgba="0.8 0.8 0.8 1.0"/>
+          </material>
+          <origin xyz="0 0 ${base_height}"/>
+          <geometry>
+            <mesh filename="package://clearpath_sensors_description/meshes/ouster/os1_base.dae"/>
+          </geometry>
+        </visual>
+        <collision>
+          <origin xyz="0 0 ${base_height/2}"/>
+          <geometry>
+            <box size="${base_length} ${base_length} ${base_height}"/>
+          </geometry>
+        </collision>
     </link>
+  </xacro:if>
+  <xacro:unless value="${base == 'base'}">
+    <link name="${name}_base_link" />
+  </xacro:unless>
     <!-- Lidar Link -->
     <link name="${name}_link">
