Commit message: Add Seyond description with lower-than-reality resolution & correct FoV for simulation. Fix math for calculating the number of samples

File: clearpath_sensors_description/urdf/seyond_lidar.urdf.xacro (robot description, xacro)
@@ -53,6 +53,6 @@
             <origin xyz="0 0 0.042" rpy="0 0 0" />
         </joint>
-        <xacro:property name="samples_h" value="${round((max_ang_h - min_ang_h) * 180 / (ang_res_h * pi))}"/>
-        <xacro:property name="samples_v" value="${round((max_ang_v - min_ang_v) * 180 / (ang_res_v * pi))}"/>
+        <xacro:property name="samples_h" value="${round((max_ang_h - min_ang_h) / ang_res_h)}"/>
+        <xacro:property name="samples_v" value="${round((max_ang_v - min_ang_v) / ang_res_v)}"/>
         <gazebo reference="${name}_laser">
             <sensor name="${name}" type="gpu_lidar">
